File: Microcontroller.sch (KiCad schematic (older format))
At the start: 12 parts, among them U7 STM32F103C8Tx, Y1 CRYSTAL_8MHz

Commit message: Finished rev4
Parts:
- C10, C11, C12, C13, C5, C6, C9: footprint Capacitors_SMD:C_0603 -> Capacitors_SMD:C_0805_HandSoldering
- C7, C8: value 6.8p -> 18p; footprint Capacitors_SMD:C_0603 -> Capacitors_SMD:C_0805_HandSoldering
- R19: footprint Resistors_SMD:R_0805 -> Resistors_SMD:R_0805_HandSoldering
- U7: value STM32F103C8Tx -> STM32F100C8Tx; symbol STM32F103C8Tx -> STM32F100C8Tx
- Y1: footprint Crystals:HC-33UV -> Crystals:Crystal_HC49-U_Vertical
Connections:
- net UART1_RE: now reaches U7.17 (ADC1_IN7/SPI1_MOSI/TIM17_CH1/TIM1_CH1N/TIM3_CH2/PA7)
- net BUTTON_USER: now reaches U7.33 (TIM1_ETR/USART1_RTS/PA12)
- net TERM_ENALBE renamed TERM_ENABLE
- no-connect marks 11 -> 10
Changed lines of the file:
@@
 LIBS:stm32
 LIBS:VL53L0X
+LIBS:mechanical
+LIBS:switches
 LIBS:sensorGridPcb-cache
 EELAYER 26 0
@@
 $EndDescr
 $Comp
-L STM32F103C8Tx U7
+L STM32F100C8Tx U7
 U 1 1 582DAACC
 P 6000 3750
-F 0 "U7" H 4800 5500 50  0000 C CNN
-F 1 "STM32F103C8Tx" H 4800 5700 50  0000 C CNN
-F 2 "Housings_QFP:LQFP-48_7x7mm_Pitch0.5mm" H 4800 5600 50  0000 C CNN
+F 0 "U7" H 6000 5818 50  0000 C CNN
+F 1 "STM32F100C8Tx" H 4750 5750 50  0000 C CNN
+F 2 "Housings_QFP:LQFP-48_7x7mm_Pitch0.5mm" H 4750 5600 50  0000 C CNN
 F 3 "" H 6000 3750 50  0000 C CNN
 	1    6000 3750
@@
 F 0 "C10" V 6800 1750 50  0000 L CNN
 F 1 "100n" V 6700 1750 50  0000 L CNN
-F 2 "Capacitors_SMD:C_0603" H 6788 1550 50  0001 C CNN
+F 2 "Capacitors_SMD:C_0805_HandSoldering" H 6788 1550 50  0001 C CNN
 F 3 "" H 6750 1700 50  0000 C CNN
 	1    6750 1700
@@
 F 0 "C13" V 6800 1000 50  0000 L CNN
 F 1 "100n" V 6700 1000 50  0000 L CNN
-F 2 "Capacitors_SMD:C_0603" H 6788 800 50  0001 C CNN
+F 2 "Capacitors_SMD:C_0805_HandSoldering" H 6788 800 50  0001 C CNN
 F 3 "" H 6750 950 50  0000 C CNN
 	1    6750 950
@@
 F 0 "C12" V 6800 1250 50  0000 L CNN
 F 1 "100n" V 6700 1250 50  0000 L CNN
-F 2 "Capacitors_SMD:C_0603" H 6788 1050 50  0001 C CNN
+F 2 "Capacitors_SMD:C_0805_HandSoldering" H 6788 1050 50  0001 C CNN
 F 3 "" H 6750 1200 50  0000 C CNN
 	1    6750 1200
@@
 F 0 "C9" V 6800 2050 50  0000 L CNN
 F 1 "1u" V 6700 2050 50  0000 L CNN
-F 2 "Capacitors_SMD:C_0603" H 6788 1800 50  0001 C CNN
+F 2 "Capacitors_SMD:C_0805_HandSoldering" H 6788 1800 50  0001 C CNN
 F 3 "" H 6750 1950 50  0000 C CNN
 	1    6750 1950
@@
 F 0 "C5" V 2148 2050 50  0000 C CNN
 F 1 "1u" V 2239 2050 50  0000 C CNN
-F 2 "Capacitors_SMD:C_0603" H 2438 1900 50  0001 C CNN
+F 2 "Capacitors_SMD:C_0805_HandSoldering" H 2438 1900 50  0001 C CNN
 F 3 "" H 2400 2050 50  0000 C CNN
 	1    2400 2050
@@
 F 0 "Y1" V 1896 3312 50  0000 R CNN
 F 1 "CRYSTAL_8MHz" H 1650 3400 50  0000 R CNN
-F 2 "Crystals:HC-33UV" H 1850 3400 50  0001 C CNN
+F 2 "Crystals:Crystal_HC49-U_Vertical" H 1850 3400 50  0001 C CNN
 F 3 "" H 1850 3400 50  0000 C CNN
 	1    1850 3400
@@
 F 0 "R19" V 2000 3550 50  0000 C CNN
 F 1 "220" V 2100 3500 50  0000 C CNN
-F 2 "Resistors_SMD:R_0805" V 2030 3500 50  0001 C CNN
+F 2 "Resistors_SMD:R_0805_HandSoldering" V 2030 3500 50  0001 C CNN
 F 3 "" H 2100 3500 50  0000 C CNN
 	1    2100 3500
@@
 P 1550 3300
 F 0 "C7" V 1802 3300 50  0000 C CNN
-F 1 "6.8p" V 1711 3300 50  0000 C CNN
-F 2 "Capacitors_SMD:C_0603" H 1588 3150 50  0001 C CNN
+F 1 "18p" V 1711 3300 50  0000 C CNN
+F 2 "Capacitors_SMD:C_0805_HandSoldering" H 1588 3150 50  0001 C CNN
 F 3 "" H 1550 3300 50  0000 C CNN
 	1    1550 3300
@@
 P 1550 3500
 F 0 "C8" V 1400 3500 50  0000 C CNN
-F 1 "6.8p" V 1300 3500 50  0000 C CNN
-F 2 "Capacitors_SMD:C_0603" H 1588 3350 50  0001 C CNN
+F 1 "18p" V 1300 3500 50  0000 C CNN
+F 2 "Capacitors_SMD:C_0805_HandSoldering" H 1588 3350 50  0001 C CNN
 F 3 "" H 1550 3500 50  0000 C CNN
 	1    1550 3500
@@
 	2900 1850 2900 2350
 Wire Wire Line
-	2900 2350 3100 2350
+	2900 2350 3300 2350
 Wire Wire Line
 	2750 2250 2750 2550
 Wire Wire Line
-	2750 2550 3100 2550
+	2750 2550 3300 2550
 $Comp
 L C C6
@@
 F 0 "C6" V 1948 2800 50  0000 C CNN
 F 1 "100n" V 2039 2800 50  0000 C CNN
-F 2 "Capacitors_SMD:C_0603" H 2238 2650 50  0001 C CNN
+F 2 "Capacitors_SMD:C_0805_HandSoldering" H 2238 2650 50  0001 C CNN
 F 3 "" H 2200 2800 50  0000 C CNN
 	1    2200 2800
@@
 	2550 3300 2550 2950
 Wire Wire Line
-	2550 2950 3100 2950
-Wire Wire Line
-	3100 3050 2650 3050
+	2550 2950 3300 2950
+Wire Wire Line
+	2650 3050 3300 3050
 Wire Wire Line
 	2650 3050 2650 3500
@@
 	2650 3500 2250 3500
 $Comp
-L +3.3V #PWR034
+L +3.3V #PWR048
 U 1 1 582EC6F5
 P 2500 2700
-F 0 "#PWR034" H 2500 2550 50  0001 C CNN
+F 0 "#PWR048" H 2500 2550 50  0001 C CNN
 F 1 "+3.3V" H 2515 2873 50  0000 C CNN
 F 2 "" H 2500 2700 50  0000 C CNN
@@
 	2850 2800 2850 2750
 Wire Wire Line
-	2850 2750 3100 2750
+	2850 2750 3300 2750
 Connection ~ 2500 2800
 Text HLabel 2950 4250 0    60   Output ~ 0
@@
 I2C_SDA
 Wire Wire Line
-	2950 4250 3100 4250
-Wire Wire Line
-	2950 4350 3100 4350
+	2950 4250 3300 4250
+Wire Wire Line
+	2950 4350 3300 4350
 Text HLabel 9050 3950 2    60   Input ~ 0
 UART2_RX
@@
 UART2_TX
 Wire Wire Line
-	8900 3850 9050 3850
-Wire Wire Line
-	8900 3950 9050 3950
+	8700 3850 9050 3850
+Wire Wire Line
+	8700 3950 9050 3950
 Text HLabel 9050 4450 2    60   Output ~ 0
 UART1_DE
@@
 UART1_RX
 Wire Wire Line
-	9050 4550 8900 4550
-Wire Wire Line
-	8900 4650 9050 4650
-Wire Wire Line
-	8900 4450 9050 4450
+	8700 4550 9050 4550
+Wire Wire Line
+	8700 4650 9050 4650
+Wire Wire Line
+	8700 4450 9050 4450
 Text HLabel 2900 1850 1    60   Input ~ 0
 NRST
@@
 SWD_CLK
 Wire Wire Line
-	8900 5050 9050 5050
-Wire Wire Line
-	9050 4950 8900 4950
+	8700 5050 9050 5050
+Wire Wire Line
+	8700 4950 9050 4950
 Text HLabel 9050 3750 2    60   Input ~ 0
 ADDRESS_IN_A
@@
 ADDRESS_OUT_A
 Wire Wire Line
-	9050 3650 8900 3650
-Wire Wire Line
-	8900 3750 9050 3750
+	8700 3650 9050 3650
+Wire Wire Line
+	8700 3750 9050 3750
 Text HLabel 2900 4950 0    60   Output ~ 0
 LED_STATUS
@@
 LED_TX
 Wire Wire Line
-	2900 5050 3100 5050
-Wire Wire Line
-	3100 5150 2900 5150
-Wire Wire Line
-	2900 4950 3100 4950
-NoConn ~ 3100 3250
-NoConn ~ 3100 3350
-NoConn ~ 3100 3450
-NoConn ~ 3100 3850
-NoConn ~ 3100 4450
-NoConn ~ 3100 4550
-NoConn ~ 8900 4250
-NoConn ~ 8900 4350
-NoConn ~ 8900 4850
-NoConn ~ 8900 5150
+	2900 5050 3300 5050
+Wire Wire Line
+	2900 5150 3300 5150
+Wire Wire Line
+	2900 4950 3300 4950
+NoConn ~ 3300 3250
+NoConn ~ 3300 3350
+NoConn ~ 3300 3450
+NoConn ~ 3300 3850
+NoConn ~ 3300 4450
+NoConn ~ 3300 4550
+NoConn ~ 8700 4250
+NoConn ~ 8700 5150
 Text HLabel 2950 3750 0    60   Output ~ 0
 VL53L0X_A_XSHUT
@@
 VL53L0X_A_GPIO1
 $Comp
-L VSS #PWR035
+L VSS #PWR049
 U 1 1 583909E0
 P 1200 3600
-F 0 "#PWR035" H 1200 3450 50  0001 C CNN
+F 0 "#PWR049" H 1200 3450 50  0001 C CNN
 F 1 "VSS" H 1218 3773 50  0000 C CNN
 F 2 "" H 1200 3600 50  0000 C CNN
@@
 $EndComp
 $Comp
-L VSS #PWR036
+L VSS #PWR050
 U 1 1 58390A9E
 P 1900 2200
-F 0 "#PWR036" H 1900 2050 50  0001 C CNN
+F 0 "#PWR050" H 1900 2050 50  0001 C CNN
 F 1 "VSS" H 1918 2373 50  0000 C CNN
 F 2 "" H 1900 2200 50  0000 C CNN
@@
 $EndComp
 $Comp
-L VSS #PWR037
+L VSS #PWR051
 U 1 1 58390ACD
 P 1900 2900
-F 0 "#PWR037" H 1900 2750 50  0001 C CNN
+F 0 "#PWR051" H 1900 2750 50  0001 C CNN
 F 1 "VSS" H 1918 3073 50  0000 C CNN
 F 2 "" H 1900 2900 50  0000 C CNN
@@
 $EndComp
 Wire Wire Line
-	2950 3650 3100 3650
-Wire Wire Line
-	3100 3750 2950 3750
+	2950 3650 3300 3650
+Wire Wire Line
+	2950 3750 3300 3750
 Text HLabel 2950 3950 0    60   Input ~ 0
 VL53L0X_B_GPIO1
@@
 VL53L0X_B_XSHUT
 Wire Wire Line
-	2950 3950 3100 3950
-Wire Wire Line
-	2950 4050 3100 4050
+	2950 3950 3300 3950
+Wire Wire Line
+	2950 4050 3300 4050
 Text HLabel 2900 4650 0    60   Output ~ 0
 VL53L0X_C_XSHUT
 Wire Wire Line
-	2900 4650 3100 4650
-NoConn ~ 3100 4850
+	2900 4650 3300 4650
+NoConn ~ 3300 4850
 Text HLabel 2950 4150 0    60   Input ~ 0
 VL53L0X_C_GPIO1
 Wire Wire Line
-	2950 4150 3100 4150
+	2950 4150 3300 4150
 Text HLabel 9050 4750 2    60   Output ~ 0
-TERM_ENALBE
-Wire Wire Line
-	8900 4750 9050 4750
-$Comp
-L VSS #PWR038
+TERM_ENABLE
+Wire Wire Line
+	8700 4750 9050 4750
+$Comp
+L VSS #PWR052
 U 1 1 583C1815
 P 5950 5750
-F 0 "#PWR038" H 5950 5600 50  0001 C CNN
+F 0 "#PWR052" H 5950 5600 50  0001 C CNN
 F 1 "VSS" H 5968 5923 50  0000 C CNN
 F 2 "" H 5950 5750 50  0000 C CNN
@@
 F 0 "C11" V 6800 1500 50  0000 L CNN
 F 1 "100n" V 6700 1500 50  0000 L CNN
-F 2 "Capacitors_SMD:C_0603" H 6788 1300 50  0001 C CNN
+F 2 "Capacitors_SMD:C_0805_HandSoldering" H 6788 1300 50  0001 C CNN
 F 3 "" H 6750 1450 50  0000 C CNN
 	1    6750 1450
@@
 	7000 950  7000 1950
 $Comp
-L +3.3V #PWR039
+L +3.3V #PWR053
 U 1 1 583B354E
 P 5700 1200
-F 0 "#PWR039" H 5700 1050 50  0001 C CNN
+F 0 "#PWR053" H 5700 1050 50  0001 C CNN
 F 1 "+3.3V" H 5715 1373 50  0000 C CNN
 F 2 "" H 5700 1200 50  0000 C CNN
@@
 $EndComp
 $Comp
-L VSS #PWR040
+L VSS #PWR054
 U 1 1 583B3A50
 P 7600 1600
-F 0 "#PWR040" H 7600 1450 50  0001 C CNN
+F 0 "#PWR054" H 7600 1450 50  0001 C CNN
 F 1 "VSS" H 7618 1773 50  0000 C CNN
 F 2 "" H 7600 1600 50  0000 C CNN
@@
 ADDRESS_OUT_B
 Wire Wire Line
-	9050 4050 8900 4050
-Wire Wire Line
-	8900 4150 9050 4150
+	8700 4050 9050 4050
+Wire Wire Line
+	8700 4150 9050 4150
+NoConn ~ 3300 4750
+Text HLabel 9050 4850 2    60   Input ~ 0
+BUTTON_USER
+Wire Wire Line
+	9050 4850 8700 4850
+Text HLabel 9050 4350 2    60   Output ~ 0
+UART1_RE
+Wire Wire Line
+	9050 4350 8700 4350
 $EndSCHEMATC
