File: sensorGridPcb.kicad_pcb (KiCad board)
At the start: 2 copper layers, 100 x 50 mm, 62 parts, among them J1 RJ45_A, J2 RJ45_B, P1 CONN_SWD, P2 CONN_DEBUG, U1 PC827, U10 VL53L0X, U2 PC827, U3 ST1480ACDR, U5 CRE1S1205SC, U6 LD1117S33CTR, U7 STM32F103C8Tx, U8 VL53L0X, U9 VL53L0X, Y1 CRYSTAL_8MHz

Commit message: Finished rev4
Parts:
- added C20: NM, Capacitors_SMD:CP_Elec_5x5.7, F.Cu at (92.0, 78.8)
- added C21: 100n, Capacitors_SMD:C_0805_HandSoldering, F.Cu at (120.5, 79.8)
- added J3: CONN_UART1, Pin_Headers:Pin_Header_Straight_1x03_Pitch2.54mm, F.Cu at (85.3, 74.8)
- added J4: CONN_A, Socket_Strips:Socket_Strip_Straight_1x05_Pitch2.54mm, F.Cu at (44.0, 72.0)
- added J5: CONN_B, Socket_Strips:Socket_Strip_Straight_1x05_Pitch2.54mm, F.Cu at (136.2, 44.2)
- added J6: CONN_SAT_A, Pin_Headers:Pin_Header_Straight_2x05_Pitch2.54mm, B.Cu at (70.6, 57.0)
- added J7: CONN_SAT_B, Pin_Headers:Pin_Header_Straight_2x05_Pitch2.54mm, B.Cu at (108.8, 67.3)
- added R32: 220, Resistors_SMD:R_0805_HandSoldering, F.Cu at (114.3, 45.0)
- added REF**: MountingHole_3mm, Mounting_Holes:MountingHole_3mm, F.Cu at (102.0, 66.0)
- added REF**: MountingHole_3mm, Mounting_Holes:MountingHole_3mm, F.Cu at (136.0, 82.0)
- added REF**: MountingHole_3mm, Mounting_Holes:MountingHole_3mm, F.Cu at (44.0, 44.0)
- added REF**: Fiducial_1mm_Dia_2.54mm_Outer_CopperTop, Fiducials:Fiducial_1mm_Dia_2.54mm_Outer_CopperTop, F.Cu at (137.0, 75.0)
- added REF**: Fiducial_1mm_Dia_2.54mm_Outer_CopperTop, Fiducials:Fiducial_1mm_Dia_2.54mm_Outer_CopperTop, F.Cu at (49.0, 48.0)
- added REF***: ESD-Logo_6.6x6mm_SilkScreen, Symbols:ESD-Logo_6.6x6mm_SilkScreen, F.Cu at (84.0, 62.8)
- added SW1: SW_RESET, Buttons_Switches_ThroughHole:SW_PUSH_SMALL, F.Cu at (98.7, 45.3)
- added SW2: SW_USER, Buttons_Switches_ThroughHole:SW_PUSH_SMALL, F.Cu at (108.6, 45.3)
- added TP1: TP_ADDRESS_IN_A, Measurement_Points:Measurement_Point_Round-SMD-Pad_Small, F.Cu at (58.0, 55.3)
- added TP2: TP_ADDRESS_OUT_A, Measurement_Points:Measurement_Point_Round-SMD-Pad_Small, F.Cu at (45.3, 53.3)
- added TP3: TP_ADDRESS_A, Measurement_Points:Measurement_Point_Round-SMD-Pad_Small, F.Cu at (58.3, 51.3)
- added TP4: TP_ADDRESS_IN_B, Measurement_Points:Measurement_Point_Round-SMD-Pad_Small, F.Cu at (126.0, 76.0)
- added TP5: TP_UART1_DE, Measurement_Points:Measurement_Point_Round-SMD-Pad_Small, F.Cu at (76.5, 67.3)
- added TP6: TP_ADDRESS_OUT_B, Measurement_Points:Measurement_Point_Round-SMD-Pad_Small, F.Cu at (130.0, 76.0)
- added TP7: TP_ADDRESS_B, Measurement_Points:Measurement_Point_Round-SMD-Pad_Small, F.Cu at (134.0, 76.0)
- added TP9: TP_UART1_RE, Measurement_Points:Measurement_Point_Round-SMD-Pad_Small, F.Cu at (78.8, 67.3)
- added TP_3V3: TP_3.3v, Measurement_Points:Measurement_Point_Round-SMD-Pad_Small, F.Cu at (111.0, 53.8)
- added TP_VSS: TP_VSS, Measurement_Points:Measurement_Point_Round-SMD-Pad_Small, F.Cu at (111.0, 51.3)
- added U4: CPC1017N, modlib:CPC1017N, F.Cu at (64.7, 79.0)
- C1, C10, C11, C12, C13, C14, C15, C16, C17, C18, C19, C2, C3, C4, C5, C6, C9: footprint Capacitors_SMD:C_0603 -> Capacitors_SMD:C_0805_HandSoldering
- C7, C8: value 10p -> 18p; footprint Capacitors_SMD:C_0603 -> Capacitors_SMD:C_0805_HandSoldering
- D1: value LED_TERM -> TERM
- D2: value LED_STATUS -> STAT
- D3: value LED_RX -> RX
- D4: value LED_TX -> TX
- R1, R5: value R -> 470; footprint Resistors_SMD:R_0805 -> Resistors_SMD:R_0805_HandSoldering
- R10, R4: value ? -> 220; footprint Resistors_SMD:R_0805 -> Resistors_SMD:R_0805_HandSoldering
- R11, R13, R14, R15, R16, R17, R18, R19, R2, R20, R21, R22, R23, R24, R25, R3, R6, R7, R8: footprint Resistors_SMD:R_0805 -> Resistors_SMD:R_0805_HandSoldering
- R12: value R -> 1k; footprint Resistors_SMD:R_0805 -> Resistors_SMD:R_0805_HandSoldering
- U1, U2: value PC827 -> LTV-207; footprint Housings_DIP:DIP-8_W7.62mm -> modlib:SOP8
- U10: value VL53L0X -> VL53L0X_C
- U3: value ST1480ACDR -> MAX3075E; footprint Housings_SOIC:SOIC-8_3.9x4.9mm_Pitch1.27mm -> Housings_DIP:DIP-8_W7.62mm_Socket
- U7: value STM32F103C8Tx -> STM32F100C8Tx
- U8: value VL53L0X -> VL53L0X_A
- U9: value VL53L0X -> VL53L0X_B
- Y1: footprint Crystals:HC-33UV -> Crystals:Crystal_HC49-U_Vertical
- moved C14 217.6 mm to (64.0, 61.0)
- moved C15 211.6 mm to (64.0, 59.0)
- moved R4 205.3 mm to (47.8, 54.2), turned to 270 degrees
- moved R2 199.6 mm to (50.0, 54.2), turned to 270 degrees
- moved R20 199.4 mm to (65.0, 71.8)
- moved R21 196.0 mm to (65.1, 69.8)
- moved R3 191.8 mm to (54.5, 54.2), turned to 90 degrees
- moved R1 190.9 mm to (52.3, 54.2), turned to 270 degrees
- moved C17 188.4 mm to (90.0, 58.8)
- moved C16 181.9 mm to (90.0, 61.0)
- moved R23 179.3 mm to (89.5, 68.8), turned to 180 degrees
- moved R12 176.9 mm to (65.0, 73.7), turned to 180 degrees
- moved C7 169.9 mm to (67.5, 47.2), turned to 270 degrees
- moved R22 169.2 mm to (89.5, 70.8), turned to 180 degrees
- moved C8 168.9 mm to (69.5, 52.5), turned to 90 degrees
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Connections:
- C14 pad 1: Net-(C14-Pad1) -> +3V3
- C15 pad 1: Net-(C14-Pad1) -> +3V3
- C16 pad 1: Net-(C16-Pad1) -> +3V3
- C17 pad 1: Net-(C16-Pad1) -> +3V3
- C18 pad 1: Net-(C18-Pad1) -> +3V3
- C19 pad 1: Net-(C18-Pad1) -> +3V3
- J1 pad 1: +12V -> /RS485+
- J1 pad 2: +12V -> /RS485-
- J1 pad 4: /RS485+ -> +12V
- J1 pad 5: /RS485- -> +12V
- J2 pad 1: +12V -> /RS485+
- J2 pad 2: +12V -> /RS485-
- J2 pad 4: /RS485+ -> +12V
- J2 pad 5: /RS485- -> +12V
- R11 pad 1: /RS485+ -> /RS485-
- R3 pad 1: Net-(J1-Pad3) -> +12V
- R3 pad 2: +12V -> Net-(J1-Pad3)
- R6 pad 2: /RS485- -> /RS485+
- R8 pad 1: Net-(J2-Pad3) -> +12V
- R8 pad 2: +12V -> Net-(J2-Pad3)
- R9 pad 2: /RS485- -> /RS485+
- U10 pad 1: Net-(C18-Pad1) -> +3V3
- U10 pad 11: Net-(C18-Pad1) -> +3V3
- U3 pad 2: /Microcontroller/UART1_DE -> /Microcontroller/UART1_RE
- U7 pad 17: Net-(U7-Pad17) -> /Microcontroller/UART1_RE
- U7 pad 33: Net-(U7-Pad33) -> /Microcontroller/BUTTON_USER
- U8 pad 1: Net-(C14-Pad1) -> +3V3
- U8 pad 11: Net-(C14-Pad1) -> +3V3
- U9 pad 1: Net-(C16-Pad1) -> +3V3
- U9 pad 11: Net-(C16-Pad1) -> +3V3
Routing:
- net /RS485-: track 0.00 -> 164.4 mm, vias 0 -> 2
- net /RS485+: track 0.00 -> 160.3 mm, vias 0 -> 2
- net VSS: track 25.7 -> 154.1 mm, vias 3 -> 30
- net /sensors/I2C_CLK: track 0.00 -> 107.4 mm, vias 0 -> 6
- net /Microcontroller/I2C_SDA: track 0.00 -> 98.3 mm, vias 0 -> 5
- net +3V3: track 24.4 -> 116.6 mm, vias 0 -> 52
- net /ADDRESS_OUT_B: track 0.00 -> 90.3 mm, vias 0 -> 4
- net +12V: track 123.4 -> 38.4 mm, vias 0 -> 2
- net GND: track 123.6 -> 44.8 mm, vias 0 -> 3
- net /RS485_TERM_ENABLE: track 0.00 -> 74.4 mm, vias 0 -> 4
- net Net-(J1-Pad3): track 0.00 -> 66.7 mm
- net /ADDRESS_IN_B: track 0.00 -> 64.2 mm, vias 0 -> 6
- net /Microcontroller/VL53L0X_C_XSHUT: track 0.00 -> 55.8 mm, vias 0 -> 3
- net /Microcontroller/VL53L0X_C_GPIO1: track 0.00 -> 52.5 mm, vias 0 -> 3
- net Net-(J2-Pad3): track 0.00 -> 52.3 mm
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- added copper zone on In1.Cu, net +12V
- added copper zone on B.Cu, net +3V3
- added copper zone on In1.Cu, net +3V3
- added copper zone on In2.Cu, net GND
- added copper zone on In2.Cu, net VSS
- removed copper zone on B.Cu, net VSS
Other:
- board size 100 x 50 mm -> 100 x 46 mm
- copper layers 2 -> 4
- net class Power added: clearance 0.5, trace_width 0.25, via_dia 0.8, via_drill 0.4
- net class RS485 added: clearance 0.2, trace_width 0.5, via_dia 0.8, via_drill 0.4
- rule pad_to_mask_clearance: 0.2 -> 0
- board text added: "+"
- board text added: "-"
- board text added: "20-4-2017"
- board text added: "Address"
- board text added: "Design by Martijn Stommels"
- board text added: "FHICT SensorGrid Node V1"
- board text added: "NOT ethernet. SensorGrid Only!"
- board text added: "RS485+"
- board text added: "RS485-"
- board text added: "Reset"
- board text added: "User"
