File: sensorGridPcb.sch (KiCad schematic (older format))
At the start: 36 parts, among them J1 RJ45_A, J2 RJ45_B, P1 CONN_SWD, P2 CONN_DEBUG, U1 PC827, U2 PC827, U3 ST1480ACDR, U4 CPC1017N, U5 CRE1S1205SC, U6 LD1117S33CTR

Commit message: Finished rev4
Parts:
- removed U3: ST1480ACDR, Housings_SOIC:SOIC-8_3.9x4.9mm_Pitch1.27mm, symbol 75176
- added C20: NM, Capacitors_SMD:CP_Elec_5x5.7, symbol CP1
- added C21: 100n, Capacitors_SMD:C_0805, symbol C
- added J3: CONN_UART1, Pin_Headers:Pin_Header_Straight_1x03_Pitch2.54mm, symbol CONN_01X03
- added J4: CONN_A, Socket_Strips:Socket_Strip_Straight_1x05_Pitch2.54mm, symbol CONN_01X05
- added J5: CONN_B, Socket_Strips:Socket_Strip_Straight_1x05_Pitch2.54mm, symbol CONN_01X05
- added R32: 220, Resistors_SMD:R_0805_HandSoldering, symbol R
- added SW1: SW_RESET, Buttons_Switches_ThroughHole:SW_PUSH_SMALL, symbol SW_Push
- added SW2: SW_USER, Buttons_Switches_ThroughHole:SW_PUSH_SMALL, symbol SW_Push
- added TP1: TP_ADDRESS_IN_A, Measurement_Points:Measurement_Point_Round-SMD-Pad_Small, symbol TEST
- added TP10: TP_VSS, Measurement_Points:Measurement_Point_Round-SMD-Pad_Small, symbol TEST
- added TP2: TP_ADDRESS_OUT_A, Measurement_Points:Measurement_Point_Round-SMD-Pad_Small, symbol TEST
- added TP3: TP_ADDRESS_A, Measurement_Points:Measurement_Point_Round-SMD-Pad_Small, symbol TEST
- added TP4: TP_ADDRESS_IN_B, Measurement_Points:Measurement_Point_Round-SMD-Pad_Small, symbol TEST
- added TP5: TP_UART1_DE, Measurement_Points:Measurement_Point_Round-SMD-Pad_Small, symbol TEST
- added TP6: TP_ADDRESS_OUT_B, Measurement_Points:Measurement_Point_Round-SMD-Pad_Small, symbol TEST
- added TP7: TP_ADDRESS_B, Measurement_Points:Measurement_Point_Round-SMD-Pad_Small, symbol TEST
- added TP8: TP_3.3v, Measurement_Points:Measurement_Point_Round-SMD-Pad_Small, symbol TEST
- added TP9: TP_UART1_RE, Measurement_Points:Measurement_Point_Round-SMD-Pad_Small, symbol TEST
- added U3: MAX3075E, Housings_DIP:DIP-8_W7.62mm_Socket, symbol MAX3075E
- C1, C2, C3, C4: footprint Capacitors_SMD:C_0603 -> Capacitors_SMD:C_0805_HandSoldering
- D1: value LED_TERM -> TERM
- D2: value LED_STATUS -> STAT
- D3: value LED_RX -> RX
- D4: value LED_TX -> TX
- R1, R5: value R -> 470; footprint Resistors_SMD:R_0805 -> Resistors_SMD:R_0805_HandSoldering
- R10, R4: value ? -> 220; footprint Resistors_SMD:R_0805 -> Resistors_SMD:R_0805_HandSoldering
- R11, R13, R14, R15, R16, R17, R18, R2, R3, R6, R7, R8: footprint Resistors_SMD:R_0805 -> Resistors_SMD:R_0805_HandSoldering
- R12: value R -> 1k; footprint Resistors_SMD:R_0805 -> Resistors_SMD:R_0805_HandSoldering
- U1, U2: value PC827 -> LTV-207; footprint Housings_DIP:DIP-8_W7.62mm -> modlib:SOP8
- U4: footprint (none) -> modlib:CPC1017N
Connections:
- net +12V: now also J1.4, J1.5, J2.4, J2.5, R3.1, R8.1, C20.1, J4.1 (P1), J5.1 (P1); no longer J1.1, J1.2, J2.1, J2.2, R3.2, R8.2
- net +3V3: now also C21.1, TP8.1, U3.8 (VCC)
- net ADDRESS_IN_A: now also TP1.1
- net ADDRESS_IN_B: now also TP4.1
- net ADDRESS_OUT_A: now also TP2.1
- net ADDRESS_OUT_B: now also TP6.1
- net GND: now also C20.2, J4.5 (P5), J5.5 (P5)
- net Microcontroller/NRST: now also SW1.1
- net Microcontroller/UART1_DE: now also TP5.1, U3.3 (DE)
- net Microcontroller/UART1_RX: now also J3.2 (P2), U3.1 (RO)
- net Microcontroller/UART1_TX: now also J3.1 (P1), U3.4 (DI)
- net RS485+: now also J1.1, J2.1, R6.2, R9.2, J4.4 (P4), J5.4 (P4), U3.6 (A); no longer J1.4, J2.4, R11.1, U4.3 (INOUT2)
- net RS485-: now also J1.2, J2.2, R11.1, U4.3 (INOUT2), J4.3 (P3), J5.3 (P3), U3.7 (B); no longer J1.5, J2.5, R6.2, R9.2
- net VSS: now also C21.2, J3.3 (P3), SW1.2, SW2.2, TP10.1, U3.5 (GND)
- net at J1.3, R1.1, U1.6: now also R3.2, J4.2 (P2), TP3.1; no longer R3.1
- net at J2.3, R5.1, U2.6: now also R8.2, J5.2 (P2), TP7.1; no longer R8.1
- new net: R32.1, SW2.1
- new net Microcontroller/BUTTON_USER: R32.2
- new net Microcontroller/UART1_RE: TP9.1, U3.2 (~RE~)
Other:
- moved on the sheet: C1, C4, R11, R12, R3, R6, R9, U4
