File: sensors.sch (KiCad schematic (older format))
At the start: 15 parts, among them U10 VL53L0X, U8 VL53L0X, U9 VL53L0X

Commit message: Finished rev4
Parts:
- added J6: CONN_SAT_A, Pin_Headers:Pin_Header_Straight_2x05_Pitch2.54mm, symbol CONN_02X05
- added J7: CONN_SAT_B, Pin_Headers:Pin_Header_Straight_2x05_Pitch2.54mm, symbol CONN_02X05
- C14, C15, C16, C17, C18, C19: footprint Capacitors_SMD:C_0603 -> Capacitors_SMD:C_0805_HandSoldering
- R20, R21, R22, R23, R24, R25: footprint Resistors_SMD:R_0805 -> Resistors_SMD:R_0805_HandSoldering
- U10: value VL53L0X -> VL53L0X_C
- U8: value VL53L0X -> VL53L0X_A
- U9: value VL53L0X -> VL53L0X_B
Connections:
- net +3V3: now also C14.1, C15.1, C16.1, C17.1, C18.1, C19.1, U10.1 (AVDDVCSEL), U10.11 (AVDD), U8.1 (AVDDVCSEL), U8.11 (AVDD), U9.1 (AVDDVCSEL), U9.11 (AVDD), J6.5 (P5), J7.5 (P5)
- net I2C_CLK: now also J6.2 (P2), J7.2 (P2)
- net I2C_SDA: now also J6.4 (P4), J7.4 (P4)
- net VL53L0X_A_GPOI1: now also J6.1 (P1)
- net VL53L0X_A_XSHUT: now also J6.3 (P3)
- net VL53L0X_C_GPOI1: now also J7.1 (P1)
- net VL53L0X_C_XSHUT: now also J7.3 (P3)
- net VSS: now also J6.6 (P6), J7.6 (P6)
- no-connect marks 3 -> 11
